File: kicad/TLS_Pie.kicad_sch (KiCad schematic)
At the start: 20 parts, among them M1 stepper + 50:1, U1 DS3231 breakout, U10 fan 5 V, U11 INA226 R002 -- NOT FITTED, U3 LM2596S-ADJ -> 5.1 V, U4 Big Easy Driver, U7 VLP-16 interface box, U8 Velodyne VLP-16

Commit message: Rev 3.1: the pack is 4S3P, the BMS was right, and every trace is now drawn
Two changes, both from the user.

FIRST: the pack is 4S3P -- 12 cells in 4 rows of 3, not the 36 that "3S12P"
claimed. That inverts the diagnosis. At 12.22 V a 4S pack sits at 3.05 V/cell,
which is genuinely low, so the 4S board already fitted was the CORRECT part
doing its job, and the ~0.55 V body-diode reading was it working rather than
failing. The original "flat battery" conclusion was right and should never have
been struck out: the argument used to void it -- "3S12P is ~330 Wh, it could not
drain in an evening" -- rested entirely on the cell count. Twelve cells is
~130 Wh, about seven hours at the rig's ~18 W.

So the fix is a 16.8 V charge and finding the weak group, not a new BMS. The 3S
board bought by mistake must not be fitted: on a 4S pack it would put ~16.8 V on
a B3+ input rated for three cells and leave the fourth group with no protection
at all.

One thing 4S makes worse, and it is flagged on the sheet: S2 hands the VLP-16
raw pack voltage, now up to 16.8 V, where the 3S assumption capped that leg at
12.6 V. Check the sensor's input range before that switch is ever closed.

SECOND: "all traces connect, no abbreviation, all on one page." The sheet was
re-laid out so nothing is joined by name. Rails are real horizontal wires, drops
are real vertical wires, junction dots are real nodes, and a crossing without a
dot is genuinely not a connection. The ten rail names are a reading aid; delete
them all and the netlist is identical.

That made the old validator useless -- it checked labels -- so it now builds a
net tracer (union-find over wire endpoints and junctions) and asserts the design
rules by following copper: the star point reaches every ground and NOT B-, C- is
a separate node from P-, each pack tap carries exactly one wire, R_PU reaches the
driver's own VCC and not the Pi's 3V3, coil A is not coil B, and every pin is
either wired or explicitly marked no-connect.

1,784 vali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
Parts:
- removed J_LIDAR: to U7 J2 barrel, symbol TLS_Pie:Conn_2
- BMS1: value NLY-3C-V3.0 (3S, common port) -> 4S separate port; symbol TLS_Pie:BMS_3S -> TLS_Pie:BMS_4S
- BT1: value 3S12P Li-ion -> 4S3P Li-ion; symbol TLS_Pie:Batt_3S12P -> TLS_Pie:Batt_4S3P
- U11: value INA226 R002 -- NOT FITTED -> INA226 -- NOT FITTED
Connections:
- net +VBATT_MON is gone; now on net +VBATT: U11.2 (IN-)
- net GND: now also BMS1.8 (P-); no longer BMS1.6 (P-), J_CHG.2
- net at BMS1.5 (B-): now also BT1.5 (B-); no longer F1.1
- net COIL_A+: no longer names the net of M1.1 (A+), U4.13 (A1)
- net COIL_A-: no longer names the net of M1.2 (A-), U4.14 (A2)
- net COIL_B+: no longer names the net of M1.3 (B+), U4.15 (B1)
- net COIL_B-: no longer names the net of M1.4 (B-), U4.16 (B2)
- net M.DIR: no longer names the net of JP1.37 (GPIO26), R_DR.1
- net M.ENABLE: no longer names the net of JP1.33 (GPIO13), R_EN.1
- net M.STEP: no longer names the net of JP1.35 (GPIO19), R_ST.1
- net SENSOR: no longer names the net of U7.4 (TB1 1-9), U8.1 (cable)
- new net: BMS1.6 (P+), F1.1
- new net CHG-: BMS1.7 (C-), J_CHG.2
Other:
- note added: "0. CHARGE AT 16.8 V. At 12.22 V this pack sits at 3.05 V/cell and the BMS is correctly latched on under-voltage; most such boards only release once a charger is applied. Do this BEFORE judging the board. 1. Four groups -- B-/B1+, B1+/B2+, B2+/B3+, B3+/B4+ -- each ~4.2 V when full and within 50 mV of the others. THE WEAK GROUP SHOWS UP HERE, and it is the one that tripped the cutoff. 2. B- to P- s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"
- note added: "A1/A2 must be the two ends of ONE coil, B1/B2 the other. Cross them and the motor buzzes, heats and does not turn. Which way round a pair goes only reverses direction, and direction is a software setting -- do not chase it with a soldering iron. Find the pairs with a meter on continuity."
- note added: "ACCEPTANCE TEST -- CHARGE FIRST, THEN MEASURE. The order is the whole point."
- note added: "CONNECT THE TAPS IN THIS ORDER: B- B1+ B2+ B3+ B4+ The protection ICs are powered from the taps. Out of order, one stage sees most of the pack across single-cell inputs and dies silently -- leaving a board that looks fine and protects nothing. Solder all five to the pack FIRST, meter the free connector, and only then plug it in. B1+/B2+/B3+ carry milliamps -- 22-24 AWG. B4+ and B- carry the FULL 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"
- note added: "Charger: 16.8 V CC-CV for 4S Li-ion. 12.6 V is a 3S charger and will never fill this pack past about half. 13.8-14.4 V is a lead-acid unit -- harmless here at 3.45-3.6 V/cell, but it undercharges. SEPARATE PORT: its negative goes to C-, never to the star point."
- note added: "INA226 DNP: the pack lead runs straight through. Fitting it means CUTTING the +VBATT rail between these two drops and letting the shunt bridge the gap. Must be the R002 variant -- R100 is good for 0.8 A and this rig pulls ~3 A."
- note added: "R_PU is the gating item -- nothing turns until it is fitted. Every Pi GPIO floats as an input for the ~30 s the Pi takes to boot, and ENABLE is active-low. Without this the driver can sit energised through the whole of boot with nothing in control of it. It goes on the DRIVER side of R_EN and pulls up to the driver's own VCC -- not the Pi's 3V3 -- so it still holds with the Pi unplugged. Set the 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"
- note added: "S1 and S2 both hang off the fused node, in PARALLEL. S1 does NOT switch the lidar -- opening S1 kills the Pi and the motor and leaves the VLP-16 spinning on S2. *** NEW ON 4S: S2 HANDS THE VLP-16 UP TO 16.8 V *** On the old 3S assumption that leg never passed 12.6 V. CHECK THE SENSOR'S OWN INPUT RANGE before S2 is ever closed. If it will not take 16.8 V that leg needs a regulator -- the one place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"
- note added: "TLS Pie -- Rev 3.1 -- generated by kicad/make_kicad_schematic.py. Edit the script, not this file. Rev 3.0 assumed a 3S pack and was WRONG. Every conductor here is drawn: nothing is joined by name, and a crossing without a junction dot is not a connection. GPIO assignment is owned by tls_stepper.py."
- note added: "Vin from header pin 1 (3V3), NEVER pin 2 or 4. This board's I2C pull-ups reference Vin, so 5 V on Vin puts 5 V on GPIO2 and GPIO3, which are not 5 V tolerant. Check before trusting it: power the board with SDA and SCL not yet fitted and measure SDA to GND -- it must read about 3.3 V. BAT / 32K / SQW / RST: open on purpose."
- note added: "ZONE A POWER CHAIN 4S3P pack -- and the 4S BMS fitted to it was right"
- note added: "ZONE B THE PI AND ITS BUS"
- note added: "ZONE C MOTOR CHAIN M+ now sees up to 16.8 V, still inside 8-35 V"
- note removed: "*** THE STAR POINT MOVED IN REV 3.0 *** Every ground in this rig lands on BMS P-, never on the pack's B-. A return wired to B- bypasses the FETs: that load is unprotected, AND it keeps draining the pack after the BMS has cut off. EXACTLY ONE wire touches B-, and it is the one from the pack."
- note removed: "1. B- to P- must read a few MILLIvolts. ~0.55 V means both FETs are off and current is sneaking through the body diodes. That is the exact 4S symptom, and it is what strangled a healthy pack. 2. P+ to P- must equal B3+ to B- within a few mV. 3. Each group -- B- to B1+, B1+ to B2+, B2+ to B3+ -- within 50 mV of the others. 12.22 V total is 4.07 V/cell: a full, healthy pack. 4. Only then close S1, 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"
- note removed: "A1/A2 must be the two ends of ONE coil, B1/B2 the two ends of the other. Cross them and the motor buzzes, heats and does not turn. Which way round a pair goes only reverses direction, and direction is a software setting (TLSPIE_DIR_FORWARD) -- do not chase it with a soldering iron. Find the pairs with a meter on continuity, motor disconnected: one coil reads a few ohms, the other open."
- note removed: "ACCEPTANCE TEST -- the same measurement that diagnosed the 4S fault"
- note removed: "CONNECT THE TAPS IN THIS ORDER: B- then B1+ then B2+ then B3+ Out of order, the protection IC sees most of the pack across one stage and dies. Solder them to the pack FIRST, meter the connector, and only then plug it into the board. B1+ and B2+ carry milliamps -- 22-24 AWG. B3+ and B- carry the FULL pack current -- run those two thick."
- note removed: "Charger: 12.6 V CC-CV ONLY. 13.8-14.4 V open circuit is a lead-acid charger and must not touch this pack. Measure it before it is ever plugged in."
- note removed: "DNP -- ordered, never connected. Decide its position NOW: the shunt sits in series with the pack lead, so retrofitting means cutting the harness you are about to make. R002 (0.002 ohm), NOT R100 -- R100 is good for 0.8 A and this rig pulls ~3 A. 3V3 only, never 5 V, or the module's I2C pull-ups put 5 V on GPIO2/GPIO3."
- note removed: "R_PU is the gating item -- nothing turns until it is fitted. Every Pi GPIO floats as an input for the ~30 s the Pi takes to boot, and ENABLE is active-low. Without this the driver can sit energised through the whole of boot with nothing in control of it. It goes on the DRIVER side of R_EN, and pulls up to the driver's own VCC -- not the Pi's 3V3 -- so it still holds with the Pi unplugged. Set the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"
- note removed: "S1 and S2 tap the same fused node in PARALLEL. S1 does NOT switch the lidar -- opening S1 kills the Pi and the motor and leaves the VLP-16 spinning on S2."
- note removed: "STAR POINT"
- note removed: "TLS Pie -- Rev 3.0 -- generated by kicad/make_kicad_schematic.py Edit the script, not this file. Supersedes Rev 2.0 (WIRING_REV2.html). Source of truth for GPIO assignment is tls_stepper.py."
- note removed: "U6 IS DELETED IN REV 3.0. A buck needs ~1.5 V of headroom, so an LM2596 set to 12 V on a 12 V pack never regulates -- it just sags under load, which is exactly when the motor needs it. M+ now takes +VSW1 directly; the Big Easy Driver accepts 8-35 V."
- note removed: "Vin from header pin 1 (3V3), NEVER pin 2 or 4. This board's I2C pull-ups reference Vin, so 5 V on Vin puts 5 V on GPIO2 and GPIO3, which are not 5 V tolerant. Check it before you trust it: power the board with SDA and SCL not yet fitted and measure SDA to GND -- it must read about 3.3 V. BAT / 32K / SQW / RST: no connection, on purpose."
- note removed: "ZONE A POWER DISTRIBUTION Rev 3.0: the 3S BMS enters here"
- note removed: "ZONE B MOTOR CHAIN unchanged from Rev 2.0 except M+"
- note removed: "ZONE C CAPTURE, CLOCK, COOLING unchanged from Rev 2.0"
- title: TLS Pie -- Rev 3.0 wiring schematic -> TLS Pie -- Rev 3.1 wiring schematic
- moved on the sheet: F1, JP1, J_CHG, M1, R_DR, R_EN, R_PU, R_ST, S1, S2, U1, U10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

Commit message: Add the USB-C charge path: PD trigger, buck, series R, into P+ and C-
The user wants to charge over USB-C and has a 303PDSink01 PD trigger board and
LM2596S-ADJ bucks. Drawn on the sheet as J_USB -> U12 -> R_CHG -> the fused
node, returning to C-.

Three things the drawing exists to stop:

The trigger board is a FIXED-VOLTAGE SOURCE, not a charger. Its three DIP
switches select from the standard PD ladder only -- 5/9/12/15/20 V -- and three
switches also rules out PPS, which would need a button sequence or I2C. There is
no 16.8 V step, which is what a 4S Li-ion pack wants, and 20 V straight onto this
pack is 5.0 V per cell. So: set the trigger to 20 V and let the buck make 16.8 V,
and find the DIP mapping by metering VBUS with nothing connected first.

20 -> 16.8 V leaves 3.2 V of headroom. That is exactly what U6 never had -- 12 V
in, 12 V out, permanently in dropout -- so this time the buck really regulates.

The LM2596-ADJ has ONE pot: voltage only, no current limit. R_CHG (3R3 10W) is
therefore the current phase, ~1.4 A into a flat pack and tapering as it fills. A
CC/CV buck with two pots replaces it outright, so its value carries the
condition rather than hiding it in a note.

Also drawn, because it is load-bearing and invisible otherwise: a buck module is
NOT isolated, so U12's IN- and OUT- are the same copper. That is what makes the
USB-C supply's ground become C- rather than the star point, and it is the reason
not to earth the rig anywhere else while charging. The validator caught this --
it asserted J_USB's ground reaches C- and the connection was not there, because
a symbol's pins are not joined by the symbol.

1,982 validator checks, 0 failed. KiCad ERC: 0 violations.

Co-Authored-By: Claude Opus 5 <noreply@anthropic.com>
Parts:
- removed J_CHG: charge socket, symbol TLS_Pie:Conn_2
- added J_USB: PD trigger 303PDSink01 @ 20 V, symbol TLS_Pie:Conn_2
- added R_CHG: 3R3 10W (omit if U12 is CC/CV), symbol TLS_Pie:R
- added U12: charge buck -> 16.8 V, symbol TLS_Pie:LM2596_Module
Connections:
- net +VBATT: now also R_CHG.2
- net CHG-: now also J_USB.2, U12.2 (OUT-), U12.3 (IN-)
- new net: R_CHG.1, U12.1 (OUT+)
- new net: J_USB.1, U12.4 (IN+)
Other:
- note added: "CHARGE PATH -- USB-C. A 4S Li-ion pack wants 16.8 V. THE PD TRIGGER IS A FIXED-VOLTAGE SOURCE, NOT A CHARGER. Its 3-way DIP selects from 5/9/12/15/20 V only -- there is NO 16.8 V step, and 20 V straight onto this pack is 5.0 V PER CELL. Set the trigger to 20 V and let U12 make 16.8 V. 20 -> 16.8 leaves 3.2 V of headroom, so unlike the deleted U6 this buck really does regulate. Find the DIP mappin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"
- note removed: "Charger: 16.8 V CC-CV for 4S Li-ion. 12.6 V is a 3S charger and will never fill this pack past about half. 13.8-14.4 V is a lead-acid unit -- harmless here at 3.45-3.6 V/cell, but it undercharges. SEPARATE PORT: its negative goes to C-, never to the star point."

Commit message: Rev 3.2: fit the BMS and buck actually bought, and both changed the topology
The Cricklewood BMS4S is COMMON PORT -- it has no C- pad -- so charge and
discharge share P+/P-.  Rev 3.1 was drawn against the separate-port board
already fitted and gave the charger its own return node and its own rail.
That rail is now deleted, not moved: the charge return IS the star point.

Two consequences that are new, and neither is a wiring choice:

  * the charger hangs across +VBATT/GND in PARALLEL with every load, upstream
    of both switches -- so charge with S1 and S2 open, or the CC limit feeds
    the load and the CV stage never terminates cleanly;
  * the buck is not isolated, so the USB-C supply's ground is bonded to the
    WHOLE rig's ground while charging, rather than to an isolated C- node.

The second part is the charger itself.  Rev 3.1 assumed a plain LM2596-ADJ,
which has one pot (voltage only), so it carried a 3R3 10 W series resistor to
do the current phase by burning the difference.  The BCD5A has two pots,
voltage and current -- that is the whole difference between a supply and a
charger -- so R_CHG is deleted.

Verified on the bench today: the PD trigger's first DIP setting read 15.15 V,
which cannot charge this pack at all.  A buck only steps down, so U12 would
have reached ~14.5 V -- 3.6 V/cell -- and the balancer would never have
started, since it only bleeds near 4.2 V/cell.  Re-dipped, it reads 20 V.

The C- design rules were INVERTED, not deleted.  The tests now assert that the
BMS has no C- pin and that R_CHG is absent, so a later session cannot quietly
reintroduce the separate-port topology from stale notes -- which is exactly the
failure mode this project has already met once.

Tap names follow the vendor's own ladder on both parts: B- B1 B2 B3 B+ at
0 / 4.2 / 8.4 / 12.6 / 16.8 V.  The pad silkscreen is the one unverified
assumption and is flagged as such in three places.

Verified: 1912 validator checks 0 failed; KiCad ERC 0 violations; netlist
carr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
Parts:
- removed R_CHG: 3R3 10W (omit if U12 is CC/CV), symbol TLS_Pie:R
- BMS1: value 4S separate port -> BMS4S 40A common port + balance
- U12: value charge buck -> 16.8 V -> BCD5A -> 16.8 V / 1.5 A; symbol TLS_Pie:LM2596_Module -> TLS_Pie:BuckCC_Module
Connections:
- net CHG- is gone; now on net GND: BMS1.7 (P-), J_USB.2, U12.2 (OUT-), U12.3 (IN-)
- net +VBATT: now also U12.1 (OUT+)
- net GND: no longer BMS1.8 (P-)
Other:
- note added: "0. SET U12 ON THE BENCH FIRST -- 16.8 V open-circuit, then 1.5 A into a dead short through the meter. NEITHER POT MAY BE TOUCHED AFTERWARDS. With the trigger on 20 V there is now a supply on this bench that would put 5.0 V/cell on the pack, so U12 is the only thing standing between them. 1. CHARGE AT 16.8 V. At 12.22 V this pack sits at 3.05 V/cell and the BMS is correctly latched on under-voltag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"
- note added: "CHARGE PATH -- USB-C. A 4S Li-ion pack wants 16.8 V. *** THE TRIGGER MUST BE ON 20 V. 15 V CANNOT CHARGE THIS PACK. *** VERIFIED 2026-08-11: first DIP setting gave 15.15 V, re-dipped and it now reads 20 V. LABEL THE BOARD IN THAT POSITION -- it is the only one that works, and the setting is three tiny switches away from being lost. Why 15 V fails: a buck ONLY steps down, so U12 would reach at bes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"
- note added: "CONNECT THE TAPS IN THIS ORDER: B- B1 B2 B3 B+ Measured against B-, they are the voltage ladder the vendor specifies: B- = 0 V B1 = 4.2 V B2 = 8.4 V B3 = 12.6 V B+ = 16.8 V METER EACH ONE ON THE FREE CONNECTOR BEFORE PLUGGING IT IN. On a flat pack they read low and evenly spaced -- what matters is the ORDER and that no two are swapped. The protection ICs are powered from the taps. Out of order, o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"
- note added: "TLS Pie -- Rev 3.2 -- generated by kicad/make_kicad_schematic.py. Edit the script, not this file. Rev 3.0 assumed a 3S pack and was WRONG. Rev 3.2 fits the bought parts: BMS4S (COMMON PORT -- no C- pad, so the old CHG- rail is deleted and the charge return is the star point) and the BCD5A CC/CV buck (two pots, so the 3R3 series resistor is deleted). Every conductor here is drawn: nothing is joine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"
- note added: "ZONE A POWER CHAIN 4S3P pack, common-port balancing BMS, USB-C charge"
- note removed: "0. CHARGE AT 16.8 V. At 12.22 V this pack sits at 3.05 V/cell and the BMS is correctly latched on under-voltage; most such boards only release once a charger is applied. Do this BEFORE judging the board. 1. Four groups -- B-/B1+, B1+/B2+, B2+/B3+, B3+/B4+ -- each ~4.2 V when full and within 50 mV of the others. THE WEAK GROUP SHOWS UP HERE, and it is the one that tripped the cutoff. 2. B- to P- s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"
- note removed: "CHARGE PATH -- USB-C. A 4S Li-ion pack wants 16.8 V. THE PD TRIGGER IS A FIXED-VOLTAGE SOURCE, NOT A CHARGER. Its 3-way DIP selects from 5/9/12/15/20 V only -- there is NO 16.8 V step, and 20 V straight onto this pack is 5.0 V PER CELL. Set the trigger to 20 V and let U12 make 16.8 V. 20 -> 16.8 leaves 3.2 V of headroom, so unlike the deleted U6 this buck really does regulate. Find the DIP mappin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"
- note removed: "CONNECT THE TAPS IN THIS ORDER: B- B1+ B2+ B3+ B4+ The protection ICs are powered from the taps. Out of order, one stage sees most of the pack across single-cell inputs and dies silently -- leaving a board that looks fine and protects nothing. Solder all five to the pack FIRST, meter the free connector, and only then plug it in. B1+/B2+/B3+ carry milliamps -- 22-24 AWG. B4+ and B- carry the FULL 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"
- note removed: "TLS Pie -- Rev 3.1 -- generated by kicad/make_kicad_schematic.py. Edit the script, not this file. Rev 3.0 assumed a 3S pack and was WRONG. Every conductor here is drawn: nothing is joined by name, and a crossing without a junction dot is not a connection. GPIO assignment is owned by tls_stepper.py."
- note removed: "ZONE A POWER CHAIN 4S3P pack -- and the 4S BMS fitted to it was right"
- title: TLS Pie -- Rev 3.1 wiring schematic -> TLS Pie -- Rev 3.2 wiring schematic
